File: siot-node-relay/siot-node-relay.kicad_pcb (KiCad board)
At the start: 2 copper layers, 40.7 x 46.6 mm, 16 parts, among them J1 xConnect_smd, J2 xConnect_smd, J3 Screw_Terminal_5mm_01x02, J4 Screw_Terminal_5mm_01x02, K1 G6DN-1A-L-DC5, Q1 BSS84, U1 DS2413P_, U2 ADP7142ARDZ-5.0, U3 STWD100NYWY3F

Commit message: updates
Parts:
- removed Q1: BSS84, digikey-footprints:SOT-23-3
- removed R1, R2: 100K, Resistor_SMD:R_0603_1608Metric
- removed U3: STWD100NYWY3F, digikey-footprints:SOT-753
Connections:
- U1 pad 4: Net-(U1-Pad4) -> Net-(D1-Pad2)
- U1 pad 6: Net-(R1-Pad2) -> Net-(D1-Pad2)
Routing:
- net Net-(D1-Pad2): track 10.7 -> 27.7 mm
- net Net-(R1-Pad2): track 10.2 -> 0.00 mm
- net +5V: track 14.2 -> 6.81 mm
- net Net-(Q1-Pad1): track 6.23 -> 0.00 mm
- net GND: track 11.5 -> 8.16 mm, vias 15 -> 14
- net +24V: track 22.8 -> 25.7 mm
Other:
- board size 40.7 x 46.6 mm -> 37.2 x 46.6 mm
- board text added: "SIOT Relay v2"
