File: siot-node-relay/siot-node-relay.sch (KiCad schematic (older format))
At the start: 15 parts, among them J1 xConnect_smd, J2 xConnect_smd, J3 Screw_Terminal_5mm_01x03, Q1 BSS84, U1 DS2413P_, U2 ADP7142ARDZ-5.0, U3 STWD100NYWY3F

Commit message: redo relay node
Parts:
- removed J3: Screw_Terminal_5mm_01x03, TerminalBlock_Phoenix:TerminalBlock_Phoenix_PT-1,5-3-5.0-H_1x03_P5.00mm_Horizontal, symbol bec-connector:Screw_Terminal_5mm_01x03
- removed RLY1: G5LE-14_DC5, digikey-footprints:Relay_THT_G5LE-14, symbol dk_Power-Relays-Over-2-Amps:G5LE-14_DC5
- added J3, J4: Screw_Terminal_5mm_01x02, TerminalBlock_Phoenix:TerminalBlock_Phoenix_PT-1,5-2-5.0-H_1x02_P5.00mm_Horizontal, symbol bec-connector:Screw_Terminal_5mm_01x02
- added K1: G6DN-1A-L-DC5, BEC:OMRON-G6DN-1A-L, symbol bec-relay:G6DN-1A-L-DC5
Connections:
- net +24V: now also J4.1 (Pin_1)
- net +5V: now also K1.1
- net GND: now also J4.2 (Pin_2)
- net at D1.2 (A), Q1.2 (D): now also K1.2
- new net relay_1: J3.1 (Pin_1), K1.4
- new net relay_2: J3.2 (Pin_2), K1.3
Other:
- note removed: "C"
- note removed: "NC"
- note removed: "NO"
Changed lines of the file:
@@
 	2200 1650 2450 1650
-$Comp
-L dk_Power-Relays-Over-2-Amps:G5LE-14_DC5 RLY1
-U 1 1 5DB070FA
-P 5800 3850
-F 0 "RLY1" H 6128 3896 50  0000 L CNN
-F 1 "G5LE-14_DC5" H 6128 3805 50  0000 L CNN
-F 2 "digikey-footprints:Relay_THT_G5LE-14" H 6000 4050 50  0001 L CNN
-F 3 "https://omronfs.omron.com/en_US/ecb/products/pdf/en-g5le.pdf" H 6000 4150 60  0001 L CNN
-F 4 "Z1011-ND" H 6000 4250 60  0001 L CNN "Digi-Key_PN"
-F 5 "G5LE-14 DC5" H 6000 4350 60  0001 L CNN "MPN"
-F 6 "Relays" H 6000 4450 60  0001 L CNN "Category"
-F 7 "Power Relays, Over 2 Amps" H 6000 4550 60  0001 L CNN "Family"
-F 8 "https://omronfs.omron.com/en_US/ecb/products/pdf/en-g5le.pdf" H 6000 4650 60  0001 L CNN "DK_Datasheet_Link"
-F 9 "/product-detail/en/omron-electronics-inc-emc-div/G5LE-14-DC5/Z1011-ND/280371" H 6000 4750 60  0001 L CNN "DK_Detail_Page"
-F 10 "RELAY GEN PURPOSE SPDT 10A 5V" H 6000 4850 60  0001 L CNN "Description"
-F 11 "Omron Electronics Inc-EMC Div" H 6000 4950 60  0001 L CNN "Manufacturer"
-F 12 "Active" H 6000 5050 60  0001 L CNN "Status"
-	1    5800 3850
-	1    0    0    -1
-$EndComp
 $Comp
 L dk_Specialized-ICs:DS2413P_ U1
@@
 	1    0    0    -1
 $EndComp
-$Comp
-L bec-connector:Screw_Terminal_5mm_01x03 J3
-U 1 1 5DB8B2BA
-P 7200 3900
-F 0 "J3" H 7150 3700 50  0000 L CNN
-F 1 "Screw_Terminal_5mm_01x03" H 7050 4150 50  0000 L CNN
-F 2 "TerminalBlock_Phoenix:TerminalBlock_Phoenix_PT-1,5-3-5.0-H_1x03_P5.00mm_Horizontal" H 7350 4300 50  0001 C CNN
-F 3 "https://media.digikey.com/pdf/Data%20Sheets/Phoenix%20Contact%20PDFs/1935174.pdf" H 7200 3900 50  0001 C CNN
-F 4 "1935174" H 7200 4200 50  0001 C CNN "MPN"
-F 5 "Phoenix Contact" H 7250 4400 50  0001 C CNN "Manufacturer"
-	1    7200 3900
-	1    0    0    -1
-$EndComp
-Wire Wire Line
-	5900 4150 6800 4150
-Wire Wire Line
-	6800 4150 6800 3900
-Wire Wire Line
-	6800 3900 7000 3900
+Wire Wire Line
+	6900 4150 6900 3900
+Wire Wire Line
+	6900 3900 7000 3900
 Wire Wire Line
 	6000 3550 6900 3550
-Wire Wire Line
-	6900 3550 6900 4000
-Wire Wire Line
-	6900 4000 7000 4000
-Wire Wire Line
-	5800 3550 5800 3450
-Wire Wire Line
-	5800 3450 7000 3450
-Wire Wire Line
-	7000 3450 7000 3800
-Text Notes 7300 4050 0    50   ~ 0
-NC
-Text Notes 7300 3950 0    50   ~ 0
-C
-Text Notes 7300 3850 0    50   ~ 0
-NO
 Text Notes 950  3250 0    50   ~ 0
 To enable relay, host must toggle PIOA \nat least once every 1.6s, or the watchdog \nchip will disable the relay. After host stops\ntoggling WD, relay will be disabled in 1.6s.
@@
 	1    0    0    -1
 $EndComp
+$Comp
+L bec-relay:G6DN-1A-L-DC5 K1
+U 1 1 5DC9B453
+P 5800 3850
+F 0 "K1" H 6130 3896 50  0000 L CNN
+F 1 "G6DN-1A-L-DC5" H 6130 3805 50  0000 L CNN
+F 2 "BEC:OMRON-G6DN-1A-L" H 6150 3800 50  0001 L CNN
+F 3 "https://www.mouser.com/datasheet/2/307/en-g6dn-838135.pdf" H 5800 3850 50  0001 C CNN
+F 4 "G6DN-1A-L DC5" H 5800 3850 50  0001 C CNN "MPN"
+F 5 "Omron" H 5800 3850 50  0001 C CNN "Manufacturer"
+	1    5800 3850
+	1    0    0    -1
+$EndComp
+Wire Wire Line
+	6000 4150 6900 4150
+Wire Wire Line
+	6900 3550 6900 3800
+Wire Wire Line
+	6900 3800 7000 3800
+$Comp
+L bec-connector:Screw_Terminal_5mm_01x02 J3
+U 1 1 5DCA5DE2
+P 7200 3900
+F 0 "J3" H 7300 3950 50  0000 L CNN
+F 1 "Screw_Terminal_5mm_01x02" H 6950 3800 50  0000 L CNN
+F 2 "TerminalBlock_Phoenix:TerminalBlock_Phoenix_PT-1,5-2-5.0-H_1x02_P5.00mm_Horizontal" H 7350 4300 50  0001 C CNN
+F 3 "https://media.digikey.com/pdf/Data%20Sheets/Phoenix%20Contact%20PDFs/1935174.pdf" H 7200 3900 50  0001 C CNN
+F 4 "1935161 " H 7200 4200 50  0001 C CNN "MPN"
+F 5 "Phoenix Contact" H 7250 4400 50  0001 C CNN "Manufacturer"
+	1    7200 3900
+	1    0    0    -1
+$EndComp
+$Comp
+L bec-connector:Screw_Terminal_5mm_01x02 J4
+U 1 1 5DE2082B
+P 7700 2350
+F 0 "J4" H 7800 2400 50  0000 L CNN
+F 1 "Screw_Terminal_5mm_01x02" H 7650 2250 50  0000 L CNN
+F 2 "TerminalBlock_Phoenix:TerminalBlock_Phoenix_PT-1,5-2-5.0-H_1x02_P5.00mm_Horizontal" H 7850 2750 50  0001 C CNN
+F 3 "https://media.digikey.com/pdf/Data%20Sheets/Phoenix%20Contact%20PDFs/1935174.pdf" H 7700 2350 50  0001 C CNN
+F 4 "1935161 " H 7700 2650 50  0001 C CNN "MPN"
+F 5 "Phoenix Contact" H 7750 2850 50  0001 C CNN "Manufacturer"
+	1    7700 2350
+	1    0    0    -1
+$EndComp
+$Comp
+L power:+24V #PWR0115
+U 1 1 5DE211AE
+P 7450 2200
+F 0 "#PWR0115" H 7450 2050 50  0001 C CNN
+F 1 "+24V" H 7465 2373 50  0000 C CNN
+F 2 "" H 7450 2200 50  0001 C CNN
+F 3 "" H 7450 2200 50  0001 C CNN
+	1    7450 2200
+	1    0    0    -1
+$EndComp
+$Comp
+L power:GND #PWR0116
+U 1 1 5DE218EB
+P 7450 2400
+F 0 "#PWR0116" H 7450 2150 50  0001 C CNN
+F 1 "GND" H 7455 2227 50  0000 C CNN
+F 2 "" H 7450 2400 50  0001 C CNN
+F 3 "" H 7450 2400 50  0001 C CNN
+	1    7450 2400
+	1    0    0    -1
+$EndComp
+Wire Wire Line
+	7500 2250 7450 2250
+Wire Wire Line
+	7450 2250 7450 2200
+Wire Wire Line
+	7450 2400 7450 2350
+Wire Wire Line
+	7450 2350 7500 2350
+Text Label 6300 3550 0    50   ~ 0
+relay_1
+Text Label 6350 4150 0    50   ~ 0
+relay_2
 $EndSCHEMATC

Commit message: updates
Parts:
- removed Q1: BSS84, digikey-footprints:SOT-23-3, symbol dk_Transistors-FETs-MOSFETs-Single:BSS84
- removed R1, R2: 100K, Resistor_SMD:R_0603_1608Metric, symbol Device:R_US
- removed U3: STWD100NYWY3F, digikey-footprints:SOT-753, symbol dk_PMIC-Supervisors:STWD100NYWY3F
Connections:
- net at U1.4 (PIOB): now also D1.2 (A), K1.2, U1.6 (PIOA)
Other:
- note added: "Relay coil current is 38mA"
- note removed: "Relay coil current is ~80mA"
- note removed: "To enable relay, host must toggle PIOA \nat least once every 1.6s, or the watchdog \nchip will disable the relay. After host stops\ntoggling WD, relay will be disabled in 1.6s."
- note removed: "Watchdog EN has internal pulldown."
Changed lines of the file:
@@
-	1    0    0    -1
-$EndComp
-$Comp
-L dk_PMIC-Supervisors:STWD100NYWY3F U3
-U 1 1 5DB13D83
-P 4100 4750
-F 0 "U3" H 3700 4150 60  0000 L CNN
-F 1 "STWD100NYWY3F" H 3300 4250 60  0000 L CNN
-F 2 "digikey-footprints:SOT-753" H 4300 4950 60  0001 L CNN
-F 3 "http://www.st.com/content/ccc/resource/technical/document/datasheet/06/6a/b3/83/9a/c7/4f/22/CD00176077.pdf/files/CD00176077.pdf/jcr:content/translations/en.CD00176077.pdf" H 4300 5050 60  0001 L CNN
-F 4 "497-10058-1-ND" H 4300 5150 60  0001 L CNN "Digi-Key_PN"
-F 5 "STWD100NYWY3F" H 4300 5250 60  0001 L CNN "MPN"
-F 6 "Integrated Circuits (ICs)" H 4300 5350 60  0001 L CNN "Category"
-F 7 "PMIC - Supervisors" H 4300 5450 60  0001 L CNN "Family"
-F 8 "http://www.st.com/content/ccc/resource/technical/document/datasheet/06/6a/b3/83/9a/c7/4f/22/CD00176077.pdf/files/CD00176077.pdf/jcr:content/translations/en.CD00176077.pdf" H 4300 5550 60  0001 L CNN "DK_Datasheet_Link"
-F 9 "/product-detail/en/stmicroelectronics/STWD100NYWY3F/497-10058-1-ND/2175107" H 4300 5650 60  0001 L CNN "DK_Detail_Page"
-F 10 "IC WATCHDOG TIME CIRCUIT SOT23-5" H 4300 5750 60  0001 L CNN "Description"
-F 11 "STMicroelectronics" H 4300 5850 60  0001 L CNN "Manufacturer"
-F 12 "Active" H 4300 5950 60  0001 L CNN "Status"
-	1    4100 4750
-	1    0    0    -1
-$EndComp
-$Comp
-L power:+5V #PWR0108
-U 1 1 5DB168B4
-P 4100 4650
-F 0 "#PWR0108" H 4100 4500 50  0001 C CNN
-F 1 "+5V" H 4115 4823 50  0000 C CNN
-F 2 "" H 4100 4650 50  0001 C CNN
-F 3 "" H 4100 4650 50  0001 C CNN
-	1    4100 4650
-	1    0    0    -1
-$EndComp
-$Comp
-L power:GND #PWR0109
-U 1 1 5DB16EA2
-P 4200 5250
-F 0 "#PWR0109" H 4200 5000 50  0001 C CNN
-F 1 "GND" H 4205 5077 50  0000 C CNN
-F 2 "" H 4200 5250 50  0001 C CNN
-F 3 "" H 4200 5250 50  0001 C CNN
-	1    4200 5250
-	1    0    0    -1
-$EndComp
-$Comp
-L power:+5V #PWR0110
-U 1 1 5DB1862E
-P 3650 4450
-F 0 "#PWR0110" H 3650 4300 50  0001 C CNN
-F 1 "+5V" H 3665 4623 50  0000 C CNN
-F 2 "" H 3650 4450 50  0001 C CNN
-F 3 "" H 3650 4450 50  0001 C CNN
-	1    3650 4450
-	1    0    0    -1
-$EndComp
-Wire Wire Line
-	3650 4750 3650 4950
-Wire Wire Line
-	3650 4950 3800 4950
-$Comp
-L Device:R_US R1
-U 1 1 5DB19349
-P 3650 4600
-F 0 "R1" H 3718 4646 50  0000 L CNN
-F 1 "100K" H 3718 4555 50  0000 L CNN
-F 2 "Resistor_SMD:R_0603_1608Metric" V 3690 4590 50  0001 C CNN
-F 3 "~" H 3650 4600 50  0001 C CNN
-	1    3650 4600
 	1    0    0    -1
 $EndComp
@@
 Wire Wire Line
 	2950 2450 3400 2450
-$Comp
-L power:GND #PWR0112
-U 1 1 5DB374FC
-P 5600 5000
-F 0 "#PWR0112" H 5600 4750 50  0001 C CNN
-F 1 "GND" H 5605 4827 50  0000 C CNN
-F 2 "" H 5600 5000 50  0001 C CNN
-F 3 "" H 5600 5000 50  0001 C CNN
-	1    5600 5000
-	1    0    0    -1
-$EndComp
 Wire Wire Line
 	6900 4150 6900 3900
@@
 Wire Wire Line
 	6000 3550 6900 3550
-Text Notes 950  3250 0    50   ~ 0
-To enable relay, host must toggle PIOA \nat least once every 1.6s, or the watchdog \nchip will disable the relay. After host stops\ntoggling WD, relay will be disabled in 1.6s.
-Text Notes 5700 4300 0    50   ~ 0
-Relay coil current is ~80mA
+Text Notes 5700 4350 0    50   ~ 0
+Relay coil current is 38mA
 Text Notes 2950 1350 0    50   ~ 0
 Power can be 5-24V. Not sure how will the linear reg will handle\n24V so may need to swap that out later for something better.
-Connection ~ 3650 4950
-Text Notes 3400 5650 0    50   ~ 0
-Watchdog EN has internal pulldown.
 $Comp
 L power:+5V #PWR0111
@@
 	5600 3450 5600 3500
 Wire Wire Line
-	5600 4950 5600 5000
-Wire Wire Line
 	5600 4150 5600 4200
-Wire Wire Line
-	2950 4950 3650 4950
 $Comp
 L bec-diode:RECT_50V_1A D1
@@
 Connection ~ 5600 4200
 Wire Wire Line
-	5600 4200 5600 4550
-$Comp
-L dk_Transistors-FETs-MOSFETs-Single:BSS84 Q1
-U 1 1 5DBE8CD5
-P 5600 4750
-F 0 "Q1" H 5708 4803 60  0000 L CNN
-F 1 "BSS84" H 5708 4697 60  0000 L CNN
-F 2 "digikey-footprints:SOT-23-3" H 5800 4950 60  0001 L CNN
-F 3 "https://www.onsemi.com/pub/Collateral/BSS84-D.PDF" H 5800 5050 60  0001 L CNN
-F 4 "BSS84CT-ND" H 5800 5150 60  0001 L CNN "Digi-Key_PN"
-F 5 "BSS84" H 5800 5250 60  0001 L CNN "MPN"
-F 6 "Discrete Semiconductor Products" H 5800 5350 60  0001 L CNN "Category"
-F 7 "Transistors - FETs, MOSFETs - Single" H 5800 5450 60  0001 L CNN "Family"
-F 8 "https://www.onsemi.com/pub/Collateral/BSS84-D.PDF" H 5800 5550 60  0001 L CNN "DK_Datasheet_Link"
-F 9 "/product-detail/en/on-semiconductor/BSS84/BSS84CT-ND/244297" H 5800 5650 60  0001 L CNN "DK_Detail_Page"
-F 10 "MOSFET P-CH 50V 130MA SOT-23" H 5800 5750 60  0001 L CNN "Description"
-F 11 "ON Semiconductor" H 5800 5850 60  0001 L CNN "Manufacturer"
-F 12 "Active" H 5800 5950 60  0001 L CNN "Status"
-	1    5600 4750
-	1    0    0    -1
-$EndComp
+	5600 4200 5600 4500
 Wire Wire Line
-	2950 2450 2950 4950
-$Comp
-L Device:R_US R2
-U 1 1 5DBEC52A
-P 5050 4600
-F 0 "R2" H 5118 4646 50  0000 L CNN
-F 1 "100K" H 5118 4555 50  0000 L CNN
-F 2 "Resistor_SMD:R_0603_1608Metric" V 5090 4590 50  0001 C CNN
-F 3 "~" H 5050 4600 50  0001 C CNN
-	1    5050 4600
-	1    0    0    -1
-$EndComp
-$Comp
-L power:+5V #PWR0113
-U 1 1 5DBECB8E
-P 5050 4450
-F 0 "#PWR0113" H 5050 4300 50  0001 C CNN
-F 1 "+5V" H 5065 4623 50  0000 C CNN
-F 2 "" H 5050 4450 50  0001 C CNN
-F 3 "" H 5050 4450 50  0001 C CNN
-	1    5050 4450
-	1    0    0    -1
-$EndComp
-Wire Wire Line
-	4500 4850 5050 4850
-Wire Wire Line
-	5050 4750 5050 4850
-Connection ~ 5050 4850
-Wire Wire Line
-	5050 4850 5300 4850
+	2950 2450 2950 2550
 $Comp
 L power:+24V #PWR0114
@@
 Text Label 6350 4150 0    50   ~ 0
 relay_2
+Wire Wire Line
+	2950 4500 5600 4500
+Wire Wire Line
+	2950 2550 3400 2550
+Connection ~ 2950 2550
+Wire Wire Line
+	2950 2550 2950 4500
 $EndSCHEMATC
