File: siot-node-current-clamp/siot-node-current-clamp.kicad_pcb (KiCad board)
At the start: 2 copper layers, 21.8 x 20.8 mm, 9 parts, among them J1 Conn_01x03_Female, J2 Conn_01x02_Female, J3 Conn_01x03_Female, U1 L78L05_SO8, U2 DS2438

Commit message: fix hole sizes
Parts:
- J1, J3: footprint Connector_PinHeader_1.27mm:PinHeader_1x03_P1.27mm_Vertical -> bec:xConnect
- J2: footprint Connector_PinHeader_1.27mm:PinHeader_1x02_P1.27mm_Vertical -> Connector_PinSocket_2.54mm:PinSocket_1x02_P2.54mm_Vertical
- moved J2 1.55 mm to (119.4, 52.1), turned to 270 degrees
- moved J1 1.25 mm to (109.2, 57.8)
- moved J3 1.25 mm to (127.0, 57.8)
- moved R1 1.02 mm to (123.2, 52.1)
- moved C1 0.89 mm to (126.4, 52.6)
Connections:
- J2 pad 1: GND -> Net-(J2-Pad1)
- J2 pad 2: Net-(J2-Pad2) -> GND
- R1 pad 2: Net-(J2-Pad2) -> Net-(J2-Pad1)
Routing:
- net Net-(J1-Pad2): track 45.4 -> 49.2 mm
- net Net-(J2-Pad1): track 0.00 -> 3.02 mm
- net +24V: track 33.8 -> 36.6 mm
- net Net-(J2-Pad2): track 2.29 -> 0.00 mm
- net Net-(C1-Pad1): track 8.08 -> 9.62 mm

Commit message: design updates
Parts:
- C2, C3: value 0.1uF -> 2.2uF
- J1, J3: value Conn_01x03_Female -> xConnect_smd; footprint bec:xConnect -> BEC:xConnect_smd
- J2: footprint Connector_PinSocket_2.54mm:PinSocket_1x02_P2.54mm_Vertical -> BEC:1x02_solder-pads
- U1: value L78L05_SO8 -> ADP7142AUJZ-3.3; footprint Package_SO:SOIC-8_3.9x4.9mm_P1.27mm -> Package_TO_SOT_SMD:TSOT-23-5
- moved C1 15.6 mm to (110.9, 55.1)
- moved R1 11.5 mm to (111.7, 52.7), turned to 0 degrees
- moved U1 10.8 mm to (109.3, 60.7), turned to 90 degrees
- moved C3 10.1 mm to (126.3, 57.5), turned to 0 degrees
- moved U2 8.07 mm to (125.0, 53.8)
- moved J1 6.82 mm to (116.0, 58.7)
- moved J3 6.34 mm to (120.7, 58.7)
- moved C2 5.04 mm to (109.1, 63.9), turned to 180 degrees
- moved J2 4.25 mm to (115.7, 54.3), turned to 90 degrees
Connections:
- C3 pad 1: +5V -> +3V3
- U1 pad 1: +5V -> +24V
- U1 pad 3: GND -> +24V
- U1 pad 4: Net-(U1-Pad4) -> +3V3
- U1 pad 5: Net-(U1-Pad5) -> +3V3
- U2 pad 5: +5V -> +3V3
- U2 pad 8: Net-(J1-Pad2) -> Net-(J1-PadY)
Routing:
- net Net-(J1-Pad2): track 49.2 -> 0.00 mm
- net +3V3: track 0.00 -> 26.3 mm
- net +24V: track 36.6 -> 14.3 mm
- net +5V: track 19.7 -> 0.00 mm, vias 2 -> 0
- net Net-(J1-PadY): track 0.00 -> 14.9 mm, vias 0 -> 2
- net Net-(C1-Pad1): track 9.62 -> 19.0 mm
- net GND: track 20.3 -> 12.8 mm, vias 5 -> 13
- net Net-(J2-Pad1): track 3.02 -> 3.89 mm

Commit message: fix missing route
Parts:
- C2, C3: value 2.2uF -> 2.2uF_50V
Routing:
- net +24V: track 14.3 -> 18.2 mm
Changed lines of the file:
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@@
     (thickness 1.6)
     (drawings 4)
-    (tracks 59)
+    (tracks 64)
     (zones 0)
     (modules 9)
@@
       (effects (font (size 1 1) (thickness 0.15)))
     )
-    (fp_text value 2.2uF (at 0 1.43) (layer F.Fab)
+    (fp_text value 2.2uF_50V (at 0 1.43) (layer F.Fab)
       (effects (font (size 1 1) (thickness 0.15)))
     )
@@
       (effects (font (size 1 1) (thickness 0.15)))
     )
-    (fp_text value 2.2uF (at 0 1.43) (layer F.Fab)
+    (fp_text value 2.2uF_50V (at 0 1.43) (layer F.Fab)
       (effects (font (size 1 1) (thickness 0.15)))
     )
@@
   (segment (start 110.28 63.4925) (end 109.9175 63.855) (width 0.25) (layer F.Cu) (net 3))
   (segment (start 110.28 61.965) (end 110.28 63.4925) (width 0.25) (layer F.Cu) (net 3))
+  (segment (start 108.38 61.105) (end 108.68 60.805) (width 0.25) (layer F.Cu) (net 3))
+  (segment (start 108.38 61.965) (end 108.38 61.105) (width 0.25) (layer F.Cu) (net 3))
+  (segment (start 108.68 60.805) (end 109.98 60.805) (width 0.25) (layer F.Cu) (net 3))
+  (segment (start 110.28 61.105) (end 110.28 61.965) (width 0.25) (layer F.Cu) (net 3))
+  (segment (start 109.98 60.805) (end 110.28 61.105) (width 0.25) (layer F.Cu) (net 3))
   (segment (start 114.105 54.255) (end 115.73 54.255) (width 0.25) (layer F.Cu) (net 6))
   (segment (start 112.505 52.655) (end 114.105 54.255) (width 0.25) (layer F.Cu) (net 6))

Commit message: updates
Other:
- board text added: "B"
- board text added: "W"
Changed lines of the file:
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@@
   (general
     (thickness 1.6)
-    (drawings 4)
+    (drawings 6)
     (tracks 64)
     (zones 0)
@@
     (tags "Through hole 1x03 single row")
     (attr smd)
-    (fp_text reference J2 (at 2.6 -0.2 180) (layer F.SilkS)
+    (fp_text reference J2 (at -2 -2.2 180) (layer F.SilkS)
       (effects (font (size 1 1) (thickness 0.15)))
     )
@@
     (tags capacitor)
     (attr smd)
-    (fp_text reference C1 (at 0 -1.651 180) (layer F.SilkS)
+    (fp_text reference C1 (at -0.4125 -1.651 180) (layer F.SilkS)
       (effects (font (size 1 1) (thickness 0.15)))
     )
@@
     )
   )
+  (gr_text B (at 118.93 51.855) (layer F.SilkS)
+    (effects (font (size 1 1) (thickness 0.15)))
+  )
+  (gr_text W (at 115.53 51.855) (layer F.SilkS)
+    (effects (font (size 1 1) (thickness 0.15)))
+  )
   (gr_line (start 107.188 50.292) (end 107.188 71.12) (layer Edge.Cuts) (width 0.05))

Commit message: updates
Parts:
- J2: footprint BEC:1x02_solder-pads -> BEC:1x03_solder-pads
- U1: value ADP7142AUJZ-3.3 -> ADP7142AUJZ-5.0
- moved J2 3.30 mm to (112.4, 54.4)
- moved C1 2.60 mm to (108.3, 55.2)
- moved R1 2.60 mm to (109.1, 52.8)
Connections:
- C3 pad 1: +3V3 -> +5V
- J2 pad 1: Net-(J2-Pad1) -> +5V
- J2 pad 2: GND -> Net-(J2-Pad2)
- R1 pad 2: Net-(J2-Pad1) -> Net-(J2-Pad2)
- U1 pad 4: +3V3 -> +5V
- U1 pad 5: +3V3 -> +5V
- U2 pad 5: +3V3 -> +5V
Routing:
- net +5V: track 0.00 -> 29.3 mm
- net +3V3: track 26.3 -> 0.00 mm
- net Net-(J2-Pad2): track 0.00 -> 8.07 mm
- net Net-(J2-Pad1): track 3.89 -> 0.00 mm
- net Net-(C1-Pad1): track 19.0 -> 21.6 mm
Other:
- board text added: "R"
- board text added: "SIOT Curr Pres v2"
