File: siot-node-current-clamp/siot-node-current-clamp.sch (KiCad schematic (older format))
At the start: 9 parts, among them J1 Conn_01x03_Female, J2 Conn_01x02_Female, J3 Conn_01x03_Female, U1 L78L05_SO8, U2 DS2438

Commit message: fix hole sizes
Parts:
- J1, J3: footprint Connector_PinHeader_1.27mm:PinHeader_1x03_P1.27mm_Vertical -> bec:xConnect
- J2: footprint Connector_PinHeader_1.27mm:PinHeader_1x02_P1.27mm_Vertical -> Connector_PinSocket_2.54mm:PinSocket_1x02_P2.54mm_Vertical
Other:
- moved on the sheet: J2
Changed lines of the file:
@@
 F 0 "J1" H 3192 3793 50  0000 C CNN
 F 1 "Conn_01x03_Female" H 3192 3794 50  0001 C CNN
-F 2 "Connector_PinHeader_1.27mm:PinHeader_1x03_P1.27mm_Vertical" H 3300 3600 50  0001 C CNN
+F 2 "bec:xConnect" H 3300 3600 50  0001 C CNN
 F 3 "~" H 3300 3600 50  0001 C CNN
 	1    3300 3600
@@
 F 0 "J3" H 7778 3580 50  0000 L CNN
 F 1 "Conn_01x03_Female" H 7642 3794 50  0001 C CNN
-F 2 "Connector_PinHeader_1.27mm:PinHeader_1x03_P1.27mm_Vertical" H 7750 3600 50  0001 C CNN
+F 2 "bec:xConnect" H 7750 3600 50  0001 C CNN
 F 3 "~" H 7750 3600 50  0001 C CNN
 	1    7750 3600
@@
 L Connector:Conn_01x02_Female J2
 U 1 1 5D33B377
-P 3950 1400
-F 0 "J2" V 3842 1448 50  0000 L CNN
-F 1 "Conn_01x02_Female" V 3887 1448 50  0001 L CNN
-F 2 "Connector_PinHeader_1.27mm:PinHeader_1x02_P1.27mm_Vertical" H 3950 1400 50  0001 C CNN
-F 3 "~" H 3950 1400 50  0001 C CNN
-	1    3950 1400
+P 4050 1400
+F 0 "J2" V 3942 1448 50  0000 L CNN
+F 1 "Conn_01x02_Female" V 3987 1448 50  0001 L CNN
+F 2 "Connector_PinSocket_2.54mm:PinSocket_1x02_P2.54mm_Vertical" H 4050 1400 50  0001 C CNN
+F 3 "~" H 4050 1400 50  0001 C CNN
+	1    4050 1400
 	0    -1   -1   0
 $EndComp
@@
 L power:GND #PWR03
 U 1 1 5D33EF3B
-P 3950 1700
-F 0 "#PWR03" H 3950 1450 50  0001 C CNN
-F 1 "GND" H 3955 1527 50  0000 C CNN
-F 2 "" H 3950 1700 50  0001 C CNN
-F 3 "" H 3950 1700 50  0001 C CNN
-	1    3950 1700
-	1    0    0    -1
-$EndComp
-Wire Wire Line
-	3950 1600 3950 1700
+P 4150 1700
+F 0 "#PWR03" H 4150 1450 50  0001 C CNN
+F 1 "GND" H 4155 1527 50  0000 C CNN
+F 2 "" H 4150 1700 50  0001 C CNN
+F 3 "" H 4150 1700 50  0001 C CNN
+	1    4150 1700
+	1    0    0    -1
+$EndComp
 Wire Wire Line
 	4050 1600 4050 2250
@@
 	5350 2900 5850 2900
 Connection ~ 4800 2250
+Wire Wire Line
+	4150 1600 4150 1700
 $EndSCHEMATC

Commit message: design updates
Parts:
- removed J1, J3: Conn_01x03_Female, bec:xConnect, symbol Connector:Conn_01x03_Female
- removed U1: L78L05_SO8, Package_SO:SOIC-8_3.9x4.9mm_P1.27mm, symbol Regulator_Linear:L78L05_SO8
- added J1, J3: xConnect_smd, BEC:xConnect_smd, symbol bec-connector:xConnect_smd
- added U1: ADP7142AUJZ-3.3, Package_TO_SOT_SMD:TSOT-23-5, symbol Regulator_Linear:ADP7142AUJZ-3.3
- C2, C3: value 0.1uF -> 2.2uF
- J2: footprint Connector_PinSocket_2.54mm:PinSocket_1x02_P2.54mm_Vertical -> BEC:1x02_solder-pads
Connections:
- net labels added: +3.3V
- net labels removed: +5V
- wire segments 36 -> 42
Other:
- moved on the sheet: C3
Changed lines of the file:
@@
 EESchema Schematic File Version 4
 LIBS:siot-node-current-clamp-cache
-EELAYER 29 0
+EELAYER 30 0
 EELAYER END
 $Descr A 11000 8500
@@
 $EndComp
 $Comp
-L Connector:Conn_01x03_Female J1
-U 1 1 5D336C3C
-P 3300 3600
-F 0 "J1" H 3192 3793 50  0000 C CNN
-F 1 "Conn_01x03_Female" H 3192 3794 50  0001 C CNN
-F 2 "bec:xConnect" H 3300 3600 50  0001 C CNN
-F 3 "~" H 3300 3600 50  0001 C CNN
-	1    3300 3600
-	-1   0    0    -1
-$EndComp
-$Comp
-L Connector:Conn_01x03_Female J3
-U 1 1 5D338F35
-P 7750 3600
-F 0 "J3" H 7778 3580 50  0000 L CNN
-F 1 "Conn_01x03_Female" H 7642 3794 50  0001 C CNN
-F 2 "bec:xConnect" H 7750 3600 50  0001 C CNN
-F 3 "~" H 7750 3600 50  0001 C CNN
-	1    7750 3600
-	1    0    0    -1
-$EndComp
-$Comp
 L power:+24V #PWR01
 U 1 1 5D33AB1A
@@
 F 0 "J2" V 3942 1448 50  0000 L CNN
 F 1 "Conn_01x02_Female" V 3987 1448 50  0001 L CNN
-F 2 "Connector_PinSocket_2.54mm:PinSocket_1x02_P2.54mm_Vertical" H 4050 1400 50  0001 C CNN
+F 2 "BEC:1x02_solder-pads" H 4050 1400 50  0001 C CNN
 F 3 "~" H 4050 1400 50  0001 C CNN
 	1    4050 1400
@@
 Wire Wire Line
 	4050 1600 4050 2250
-$Comp
-L Regulator_Linear:L78L05_SO8 U1
-U 1 1 5D33BA71
-P 5550 4250
-F 0 "U1" H 5550 4492 50  0000 C CNN
-F 1 "L78L05_SO8" H 5550 4401 50  0000 C CNN
-F 2 "Package_SO:SOIC-8_3.9x4.9mm_P1.27mm" H 5650 4450 50  0001 C CIN
-F 3 "http://www.st.com/content/ccc/resource/technical/document/datasheet/15/55/e5/aa/23/5b/43/fd/CD00000446.pdf/files/CD00000446.pdf/jcr:content/translations/en.CD00000446.pdf" H 5750 4250 50  0001 C CNN
-	1    5550 4250
-	1    0    0    -1
-$EndComp
-$Comp
-L power:+5V #PWR09
-U 1 1 5D33BA77
-P 6000 4200
-F 0 "#PWR09" H 6000 4050 50  0001 C CNN
-F 1 "+5V" H 6015 4373 50  0000 C CNN
-F 2 "" H 6000 4200 50  0001 C CNN
-F 3 "" H 6000 4200 50  0001 C CNN
-	1    6000 4200
-	1    0    0    -1
-$EndComp
-Wire Wire Line
-	5850 4250 6000 4250
-Wire Wire Line
-	6000 4250 6000 4200
+Wire Wire Line
+	6400 4250 6400 4200
 $Comp
 L power:GND #PWR07
 U 1 1 5D33BA7F
-P 5550 4600
-F 0 "#PWR07" H 5550 4350 50  0001 C CNN
-F 1 "GND" H 5555 4427 50  0000 C CNN
-F 2 "" H 5550 4600 50  0001 C CNN
-F 3 "" H 5550 4600 50  0001 C CNN
-	1    5550 4600
-	1    0    0    -1
-$EndComp
-Wire Wire Line
-	5550 4550 5550 4600
+P 5750 4700
+F 0 "#PWR07" H 5750 4450 50  0001 C CNN
+F 1 "GND" H 5755 4527 50  0000 C CNN
+F 2 "" H 5750 4700 50  0001 C CNN
+F 3 "" H 5750 4700 50  0001 C CNN
+	1    5750 4700
+	1    0    0    -1
+$EndComp
+Wire Wire Line
+	5750 4650 5750 4700
 $Comp
 L power:+24V #PWR05
@@
 Wire Wire Line
 	5050 4200 5050 4250
-Wire Wire Line
-	5050 4250 5250 4250
 $Comp
 L Device:C C2
@@
 P 5050 4550
 F 0 "C2" H 5165 4596 50  0000 L CNN
-F 1 "0.1uF" H 5165 4505 50  0000 L CNN
+F 1 "2.2uF" H 5165 4505 50  0000 L CNN
 F 2 "Capacitor_SMD:C_0603_1608Metric" H 5088 4400 50  0001 C CNN
 F 3 "~" H 5050 4550 50  0001 C CNN
@@
 L Device:C C3
 U 1 1 5D33BA94
-P 6000 4550
-F 0 "C3" H 6115 4596 50  0000 L CNN
-F 1 "0.1uF" H 6115 4505 50  0000 L CNN
-F 2 "Capacitor_SMD:C_0603_1608Metric" H 6038 4400 50  0001 C CNN
-F 3 "~" H 6000 4550 50  0001 C CNN
-	1    6000 4550
+P 6400 4550
+F 0 "C3" H 6515 4596 50  0000 L CNN
+F 1 "2.2uF" H 6515 4505 50  0000 L CNN
+F 2 "Capacitor_SMD:C_0603_1608Metric" H 6438 4400 50  0001 C CNN
+F 3 "~" H 6400 4550 50  0001 C CNN
+	1    6400 4550
 	1    0    0    -1
 $EndComp
@@
 Connection ~ 5050 4250
 Wire Wire Line
-	6000 4250 6000 4400
-Connection ~ 6000 4250
+	6400 4250 6400 4400
+Connection ~ 6400 4250
 $Comp
 L power:GND #PWR06
@@
 L power:GND #PWR010
 U 1 1 5D33BAA4
-P 6000 4750
-F 0 "#PWR010" H 6000 4500 50  0001 C CNN
-F 1 "GND" H 6005 4577 50  0000 C CNN
-F 2 "" H 6000 4750 50  0001 C CNN
-F 3 "" H 6000 4750 50  0001 C CNN
-	1    6000 4750
+P 6400 4750
+F 0 "#PWR010" H 6400 4500 50  0001 C CNN
+F 1 "GND" H 6405 4577 50  0000 C CNN
+F 2 "" H 6400 4750 50  0001 C CNN
+F 3 "" H 6400 4750 50  0001 C CNN
+	1    6400 4750
 	1    0    0    -1
 $EndComp
@@
 	5050 4700 5050 4750
 Wire Wire Line
-	6000 4700 6000 4750
+	6400 4700 6400 4750
 Wire Wire Line
 	3500 3500 3650 3500
@@
 Wire Wire Line
 	6800 2600 6800 3600
-$Comp
-L power:+5V #PWR011
-U 1 1 5D343143
-P 6700 2450
-F 0 "#PWR011" H 6700 2300 50  0001 C CNN
-F 1 "+5V" H 6715 2623 50  0000 C CNN
-F 2 "" H 6700 2450 50  0001 C CNN
-F 3 "" H 6700 2450 50  0001 C CNN
-	1    6700 2450
-	1    0    0    -1
-$EndComp
 Wire Wire Line
 	6700 2450 6700 2900
@@
 Wire Wire Line
 	4150 1600 4150 1700
+$Comp
+L bec-connector:xConnect_smd J1
+U 1 1 5D69F5B9
+P 3300 3600
+F 0 "J1" H 3600 3650 50  0000 C CNN
+F 1 "xConnect_smd" H 3600 3550 50  0000 C CNN
+F 2 "BEC:xConnect_smd" H 3250 3350 50  0001 C CNN
+F 3 "~" H 3300 3600 50  0001 C CNN
+	1    3300 3600
+	-1   0    0    -1
+$EndComp
+$Comp
+L bec-connector:xConnect_smd J3
+U 1 1 5D69FF45
+P 7750 3600
+F 0 "J3" H 7850 3650 50  0000 L CNN
+F 1 "xConnect_smd" H 7850 3550 50  0000 L CNN
+F 2 "BEC:xConnect_smd" H 7700 3350 50  0001 C CNN
+F 3 "~" H 7750 3600 50  0001 C CNN
+	1    7750 3600
+	1    0    0    -1
+$EndComp
+$Comp
+L Regulator_Linear:ADP7142AUJZ-3.3 U1
+U 1 1 5D6A1134
+P 5750 4350
+F 0 "U1" H 5750 4717 50  0000 C CNN
+F 1 "ADP7142AUJZ-3.3" H 5750 4626 50  0000 C CNN
+F 2 "Package_TO_SOT_SMD:TSOT-23-5" H 5750 3950 50  0001 C CIN
+F 3 "https://www.analog.com/media/en/technical-documentation/data-sheets/ADP7142.pdf" H 5750 3850 50  0001 C CNN
+	1    5750 4350
+	1    0    0    -1
+$EndComp
+Wire Wire Line
+	5050 4250 5300 4250
+Wire Wire Line
+	6150 4350 6250 4350
+Wire Wire Line
+	6250 4350 6250 4250
+Wire Wire Line
+	6150 4250 6250 4250
+Connection ~ 6250 4250
+Wire Wire Line
+	6250 4250 6400 4250
+Wire Wire Line
+	5300 4250 5300 4450
+Wire Wire Line
+	5300 4450 5350 4450
+Connection ~ 5300 4250
+Wire Wire Line
+	5300 4250 5350 4250
+$Comp
+L power:+3.3V #PWR0101
+U 1 1 5D6A64BE
+P 6700 2450
+F 0 "#PWR0101" H 6700 2300 50  0001 C CNN
+F 1 "+3.3V" H 6715 2623 50  0000 C CNN
+F 2 "" H 6700 2450 50  0001 C CNN
+F 3 "" H 6700 2450 50  0001 C CNN
+	1    6700 2450
+	1    0    0    -1
+$EndComp
+$Comp
+L power:+3.3V #PWR0102
+U 1 1 5D6A6E0B
+P 6400 4200
+F 0 "#PWR0102" H 6400 4050 50  0001 C CNN
+F 1 "+3.3V" H 6415 4373 50  0000 C CNN
+F 2 "" H 6400 4200 50  0001 C CNN
+F 3 "" H 6400 4200 50  0001 C CNN
+	1    6400 4200
+	1    0    0    -1
+$EndComp
 $EndSCHEMATC

Commit message: update PNs on symbols
Parts:
- C2, C3: value 2.2uF -> 2.2uF_50V; footprint Capacitor_SMD:C_0603_1608Metric -> Capacitor_SMD:C_2220_5650Metric; symbol Device:C -> bec-passive:2.2uF_50V; MPN (none) -> GRM188R61H225ME11J; Manufacturer (none) -> Murata
- U1: symbol Regulator_Linear:ADP7142AUJZ-3.3 -> bec-power:ADP7142AUJZ-3.3; MPN (none) -> ADP7142AUJZ-3.3; Manufacturer (none) -> Analog Devices
Changed lines of the file:
@@
 	5050 4200 5050 4250
 $Comp
-L Device:C C2
+L bec-passive:2.2uF_50V C2
 U 1 1 5D33BA8E
 P 5050 4550
 F 0 "C2" H 5165 4596 50  0000 L CNN
-F 1 "2.2uF" H 5165 4505 50  0000 L CNN
-F 2 "Capacitor_SMD:C_0603_1608Metric" H 5088 4400 50  0001 C CNN
-F 3 "~" H 5050 4550 50  0001 C CNN
+F 1 "2.2uF_50V" H 5165 4505 50  0000 L CNN
+F 2 "Capacitor_SMD:C_2220_5650Metric" H 5088 4400 50  0001 C CNN
+F 3 "https://product.tdk.com/info/en/catalog/datasheets/mlcc_commercial_midvoltage_en.pdf" H 5050 4550 50  0001 C CNN
+F 4 "GRM188R61H225ME11J" H 5050 4550 50  0001 C CNN "MPN"
+F 5 "Murata" H 5050 4550 50  0001 C CNN "Manufacturer"
 	1    5050 4550
 	1    0    0    -1
 $EndComp
 $Comp
-L Device:C C3
+L bec-passive:2.2uF_50V C3
 U 1 1 5D33BA94
 P 6400 4550
 F 0 "C3" H 6515 4596 50  0000 L CNN
-F 1 "2.2uF" H 6515 4505 50  0000 L CNN
-F 2 "Capacitor_SMD:C_0603_1608Metric" H 6438 4400 50  0001 C CNN
-F 3 "~" H 6400 4550 50  0001 C CNN
+F 1 "2.2uF_50V" H 6515 4505 50  0000 L CNN
+F 2 "Capacitor_SMD:C_2220_5650Metric" H 6438 4400 50  0001 C CNN
+F 3 "https://product.tdk.com/info/en/catalog/datasheets/mlcc_commercial_midvoltage_en.pdf" H 6400 4550 50  0001 C CNN
+F 4 "GRM188R61H225ME11J" H 6400 4550 50  0001 C CNN "MPN"
+F 5 "Murata" H 6400 4550 50  0001 C CNN "Manufacturer"
 	1    6400 4550
 	1    0    0    -1
@@
 $EndComp
 $Comp
-L Regulator_Linear:ADP7142AUJZ-3.3 U1
+L bec-power:ADP7142AUJZ-3.3 U1
 U 1 1 5D6A1134
 P 5750 4350
@@
 F 2 "Package_TO_SOT_SMD:TSOT-23-5" H 5750 3950 50  0001 C CIN
 F 3 "https://www.analog.com/media/en/technical-documentation/data-sheets/ADP7142.pdf" H 5750 3850 50  0001 C CNN
+F 4 "ADP7142AUJZ-3.3" H 5750 4350 50  0001 C CNN "MPN"
+F 5 "Analog Devices" H 5750 4350 50  0001 C CNN "Manufacturer"
 	1    5750 4350
 	1    0    0    -1

Commit message: fix missing route
Parts:
- C2, C3: footprint Capacitor_SMD:C_2220_5650Metric -> Capacitor_SMD:C_0603_1608Metric
Changed lines of the file:
@@
 F 0 "C2" H 5165 4596 50  0000 L CNN
 F 1 "2.2uF_50V" H 5165 4505 50  0000 L CNN
-F 2 "Capacitor_SMD:C_2220_5650Metric" H 5088 4400 50  0001 C CNN
+F 2 "Capacitor_SMD:C_0603_1608Metric" H 5088 4400 50  0001 C CNN
 F 3 "https://product.tdk.com/info/en/catalog/datasheets/mlcc_commercial_midvoltage_en.pdf" H 5050 4550 50  0001 C CNN
 F 4 "GRM188R61H225ME11J" H 5050 4550 50  0001 C CNN "MPN"
@@
 F 0 "C3" H 6515 4596 50  0000 L CNN
 F 1 "2.2uF_50V" H 6515 4505 50  0000 L CNN
-F 2 "Capacitor_SMD:C_2220_5650Metric" H 6438 4400 50  0001 C CNN
+F 2 "Capacitor_SMD:C_0603_1608Metric" H 6438 4400 50  0001 C CNN
 F 3 "https://product.tdk.com/info/en/catalog/datasheets/mlcc_commercial_midvoltage_en.pdf" H 6400 4550 50  0001 C CNN
 F 4 "GRM188R61H225ME11J" H 6400 4550 50  0001 C CNN "MPN"

Commit message: updates
Parts:
- J2: footprint BEC:1x02_solder-pads -> BEC:1x03_solder-pads; symbol Connector:Conn_01x02_Female -> Connector:Conn_01x03_Female
- U1: value ADP7142AUJZ-3.3 -> ADP7142AUJZ-5.0; MPN ADP7142AUJZ-3.3 -> ADP7142AUJZ-5.0
Connections:
- net GND: now also J2.3 (Pin_3); no longer J2.2 (Pin_2)
- net at R1.2: now also J2.2 (Pin_2); no longer J2.1 (Pin_1)
- net +3V3 renamed +5V
- net +5V: now also J2.1 (Pin_1)
Changed lines of the file:
@@
 $EndComp
 $Comp
-L Connector:Conn_01x02_Female J2
+L Connector:Conn_01x03_Female J2
 U 1 1 5D33B377
 P 4050 1400
 F 0 "J2" V 3942 1448 50  0000 L CNN
 F 1 "Conn_01x02_Female" V 3987 1448 50  0001 L CNN
-F 2 "BEC:1x02_solder-pads" H 4050 1400 50  0001 C CNN
+F 2 "BEC:1x03_solder-pads" H 4050 1400 50  0001 C CNN
 F 3 "~" H 4050 1400 50  0001 C CNN
 	1    4050 1400
@@
 P 5750 4350
 F 0 "U1" H 5750 4717 50  0000 C CNN
-F 1 "ADP7142AUJZ-3.3" H 5750 4626 50  0000 C CNN
+F 1 "ADP7142AUJZ-5.0" H 5750 4626 50  0000 C CNN
 F 2 "Package_TO_SOT_SMD:TSOT-23-5" H 5750 3950 50  0001 C CIN
 F 3 "https://www.analog.com/media/en/technical-documentation/data-sheets/ADP7142.pdf" H 5750 3850 50  0001 C CNN
-F 4 "ADP7142AUJZ-3.3" H 5750 4350 50  0001 C CNN "MPN"
+F 4 "ADP7142AUJZ-5.0" H 5750 4350 50  0001 C CNN "MPN"
 F 5 "Analog Devices" H 5750 4350 50  0001 C CNN "Manufacturer"
 	1    5750 4350
@@
 	5300 4250 5350 4250
 $Comp
-L power:+3.3V #PWR0101
-U 1 1 5D6A64BE
+L power:+5V #PWR0101
+U 1 1 5DCE2702
 P 6700 2450
 F 0 "#PWR0101" H 6700 2300 50  0001 C CNN
-F 1 "+3.3V" H 6715 2623 50  0000 C CNN
+F 1 "+5V" H 6715 2623 50  0000 C CNN
 F 2 "" H 6700 2450 50  0001 C CNN
 F 3 "" H 6700 2450 50  0001 C CNN
@@
 $EndComp
 $Comp
-L power:+3.3V #PWR0102
-U 1 1 5D6A6E0B
+L power:+5V #PWR0102
+U 1 1 5DCE2A90
 P 6400 4200
 F 0 "#PWR0102" H 6400 4050 50  0001 C CNN
-F 1 "+3.3V" H 6415 4373 50  0000 C CNN
+F 1 "+5V" H 6415 4373 50  0000 C CNN
 F 2 "" H 6400 4200 50  0001 C CNN
 F 3 "" H 6400 4200 50  0001 C CNN
@@
 	1    0    0    -1
 $EndComp
+$Comp
+L power:+5V #PWR0103
+U 1 1 5E23EB01
+P 3950 1700
+F 0 "#PWR0103" H 3950 1550 50  0001 C CNN
+F 1 "+5V" H 3965 1873 50  0000 C CNN
+F 2 "" H 3950 1700 50  0001 C CNN
+F 3 "" H 3950 1700 50  0001 C CNN
+	1    3950 1700
+	-1   0    0    1
+$EndComp
+Wire Wire Line
+	3950 1600 3950 1700
 $EndSCHEMATC
