File: siot-gateway-particle/siot-gateway-particle.kicad_pcb (KiCad board)
At the start: 2 copper layers, 100 x 45.5 mm, 18 parts, among them J1 xConnect, J2 xConnect, U1 Particle_Mesh, U2 LTC3630, U3 DS2483R, U4 DS2483R

Commit message: work on SMD xConnect connections
Parts:
- J1, J2: value xConnect -> xConnect_smd; footprint BEC:xConnect -> BEC:xConnect_smd
- moved J1 2.29 mm to (122.1, 111.8)
- moved J2 2.02 mm to (152.4, 111.8)
Connections:
- U3 pad 5: Net-(J1-Pad2) -> Net-(J1-PadY)
- U4 pad 5: Net-(J2-Pad2) -> Net-(J2-PadY)
Routing:
- net Net-(J2-PadY): track 0.00 -> 20.4 mm
- net Net-(J2-Pad2): track 20.4 -> 0.00 mm
- net Net-(J1-Pad2): track 13.3 -> 0.00 mm
- net Net-(J1-PadY): track 0.00 -> 11.7 mm
- net GND: track 8.12 -> 9.72 mm
- net +24V: track 78.2 -> 79.8 mm

Commit message: updates
Routing:
- net Net-(J2-PadY): track 20.4 -> 24.1 mm
- net Net-(J1-PadY): track 11.7 -> 15.3 mm
- net +24V: track 79.8 -> 82.8 mm
- net GND: vias 9 -> 19
Changed lines of the file:
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@@
-(kicad_pcb (version 20171130) (host pcbnew "(5.1.2-1)-1")
+(kicad_pcb (version 20171130) (host pcbnew 5.1.4)
   (general
     (thickness 1.6)
     (drawings 11)
-    (tracks 117)
+    (tracks 131)
     (zones 0)
     (modules 18)
@@
   )
   (setup
-    (last_trace_width 1.9)
+    (last_trace_width 0.25)
     (user_trace_width 0.7)
     (user_trace_width 1.9)
@@
   (gr_circle (center 189.451293 84.230648) (end 191.165793 84.230648) (layer Dwgs.User) (width 0.2))
   (gr_circle (center 94.364893 112.197448) (end 96.079393 112.197448) (layer Dwgs.User) (width 0.2))
-  (segment (start 120.95 105) (end 120.6 105.35) (width 0.25) (layer F.Cu) (net 37))
-  (segment (start 121.81 105) (end 120.95 105) (width 0.25) (layer F.Cu) (net 37))
-  (segment (start 120.6 105.35) (end 120.6 107.5) (width 0.25) (layer F.Cu) (net 37))
-  (segment (start 120.6 107.5) (end 123.4 110.3) (width 0.25) (layer F.Cu) (net 37))
-  (segment (start 123.4 110.3) (end 126.1 110.3) (width 0.25) (layer F.Cu) (net 37))
-  (segment (start 126.1 110.3) (end 127.2 111.4) (width 0.25) (layer F.Cu) (net 37))
-  (segment (start 133.985 111.125) (end 133.985 112.725) (width 0.25) (layer F.Cu) (net 27))
-  (segment (start 144.26 105.05) (end 143.81 105.5) (width 0.25) (layer F.Cu) (net 38))
-  (segment (start 145.12 105.05) (end 144.26 105.05) (width 0.25) (layer F.Cu) (net 38))
-  (segment (start 143.81 105.5) (end 143.81 108.11) (width 0.25) (layer F.Cu) (net 38))
-  (segment (start 143.81 108.11) (end 145.9 110.2) (width 0.25) (layer F.Cu) (net 38))
-  (segment (start 145.9 110.2) (end 155.9 110.2) (width 0.25) (layer F.Cu) (net 38))
-  (segment (start 155.9 110.2) (end 157.2 111.5) (width 0.25) (layer F.Cu) (net 38))
-  (segment (start 157.2 111.5) (end 157.2 113) (width 0.25) (layer F.Cu) (net 38))
+  (via (at 132.08 111.76) (size 0.8) (drill 0.4) (layers F.Cu B.Cu) (net 27))
+  (via (at 162.56 111.76) (size 0.8) (drill 0.4) (layers F.Cu B.Cu) (net 27))
+  (via (at 163.576 112.776) (size 0.8) (drill 0.4) (layers F.Cu B.Cu) (net 27))
+  (via (at 161.544 112.776) (size 0.8) (drill 0.4) (layers F.Cu B.Cu) (net 27))
+  (via (at 163.576 110.744) (size 0.8) (drill 0.4) (layers F.Cu B.Cu) (net 27))
+  (via (at 161.544 110.744) (size 0.8) (drill 0.4) (layers F.Cu B.Cu) (net 27))
+  (via (at 133.096 112.776) (size 0.8) (drill 0.4) (layers F.Cu B.Cu) (net 27))
+  (via (at 131.064 112.776) (size 0.8) (drill 0.4) (layers F.Cu B.Cu) (net 27))
+  (via (at 133.096 110.744) (size 0.8) (drill 0.4) (layers F.Cu B.Cu) (net 27))
   (segment (start 131.94 76.73) (end 131.94 76.76) (width 0.25) (layer F.Cu) (net 20))
   (segment (start 131.94 76.76) (end 118 90.7) (width 0.25) (layer F.Cu) (net 20))
@@
   (segment (start 138.6 104) (end 142.4 104) (width 0.25) (layer F.Cu) (net 21))
   (segment (start 142.4 104) (end 142.5 104.1) (width 0.25) (layer F.Cu) (net 21))
+  (segment (start 133.985 111.125) (end 133.985 112.725) (width 0.25) (layer F.Cu) (net 27))
   (segment (start 166.442 78.648) (end 166.348 78.648) (width 0.25) (layer F.Cu) (net 27))
   (segment (start 164.242 78.398) (end 163.782381 78.398) (width 0.25) (layer F.Cu) (net 27))
@@
   (via (at 162.9 88) (size 0.8) (drill 0.4) (layers F.Cu B.Cu) (net 27))
   (via (at 162.9 88.9) (size 0.8) (drill 0.4) (layers F.Cu B.Cu) (net 27))
-  (segment (start 169.61 112.89) (end 169.61 85.66) (width 1.9) (layer F.Cu) (net 28))
-  (segment (start 167 115.5) (end 169.61 112.89) (width 1.9) (layer F.Cu) (net 28))
-  (segment (start 154.04 115.5) (end 167 115.5) (width 1.9) (layer F.Cu) (net 28))
-  (segment (start 152.4 113.86) (end 154.04 115.5) (width 1.9) (layer F.Cu) (net 28))
-  (segment (start 152.4 111.76) (end 152.4 113.86) (width 1.9) (layer F.Cu) (net 28))
-  (segment (start 123.12 115.5) (end 150.425 115.5) (width 1.9) (layer F.Cu) (net 28))
-  (segment (start 122.08 114.46) (end 123.12 115.5) (width 1.9) (layer F.Cu) (net 28))
-  (segment (start 122.08 111.76) (end 122.08 114.46) (width 1.9) (layer F.Cu) (net 28))
+  (via (at 131.064 110.744) (size 0.8) (drill 0.4) (layers F.Cu B.Cu) (net 27))
+  (segment (start 122.08 114.46) (end 122.08 111.76) (width 1.9) (layer F.Cu) (net 28))
+  (segment (start 123.12 115.5) (end 122.08 114.46) (width 1.9) (layer F.Cu) (net 28))
+  (segment (start 169.61 85.66) (end 169.61 112.89) (width 1.9) (layer F.Cu) (net 28))
+  (segment (start 169.61 112.89) (end 167 115.5) (width 1.9) (layer F.Cu) (net 28))
+  (segment (start 152.4 115.316) (end 152.4 111.76) (width 1.9) (layer F.Cu) (net 28))
+  (segment (start 152.584 115.5) (end 152.4 115.316) (width 1.9) (layer F.Cu) (net 28))
+  (segment (start 152.584 115.5) (end 123.12 115.5) (width 1.9) (layer F.Cu) (net 28))
+  (segment (start 167 115.5) (end 152.584 115.5) (width 1.9) (layer F.Cu) (net 28))
   (segment (start 126.6 103) (end 126.528248 102.928248) (width 0.25) (layer F.Cu) (net 29))
   (segment (start 121.2 103) (end 126.6 103) (width 0.25) (layer F.Cu) (net 29))
@@
   (segment (start 129.4 98.116317) (end 128.2 99.316317) (width 0.7) (layer F.Cu) (net 35))
   (segment (start 129.4 97.05) (end 129.4 98.116317) (width 0.7) (layer F.Cu) (net 35))
+  (segment (start 126.1 110.3) (end 127.2 111.4) (width 0.25) (layer F.Cu) (net 37))
+  (segment (start 127.08 109.3) (end 127.08 111.76) (width 0.25) (layer F.Cu) (net 37))
+  (segment (start 126.492 108.712) (end 127.08 109.3) (width 0.25) (layer F.Cu) (net 37))
+  (segment (start 120.95 105) (end 120.6 105.35) (width 0.25) (layer F.Cu) (net 37))
+  (segment (start 120.6 105.35) (end 120.6 108.408) (width 0.25) (layer F.Cu) (net 37))
+  (segment (start 121.81 105) (end 120.95 105) (width 0.25) (layer F.Cu) (net 37))
+  (segment (start 120.6 108.408) (end 120.904 108.712) (width 0.25) (layer F.Cu) (net 37))
+  (segment (start 120.904 108.712) (end 126.492 108.712) (width 0.25) (layer F.Cu) (net 37))
+  (segment (start 155.9 110.2) (end 157.2 111.5) (width 0.25) (layer F.Cu) (net 38))
+  (segment (start 157.2 111.5) (end 157.2 113) (width 0.25) (layer F.Cu) (net 38))
+  (segment (start 157.4 109.14) (end 157.4 111.76) (width 0.25) (layer F.Cu) (net 38))
+  (segment (start 143.81 108.11) (end 144.412 108.712) (width 0.25) (layer F.Cu) (net 38))
+  (segment (start 156.972 108.712) (end 157.4 109.14) (width 0.25) (layer F.Cu) (net 38))
+  (segment (start 145.12 105.05) (end 144.26 105.05) (width 0.25) (layer F.Cu) (net 38))
+  (segment (start 144.26 105.05) (end 143.81 105.5) (width 0.25) (layer F.Cu) (net 38))
+  (segment (start 143.81 105.5) (end 143.81 108.11) (width 0.25) (layer F.Cu) (net 38))
+  (segment (start 144.412 108.712) (end 156.972 108.712) (width 0.25) (layer F.Cu) (net 38))
   (zone (net 27) (net_name GND) (layer F.Cu) (hatch edge 0.508)
     (connect_pads yes (clearance 0.2032))

Commit message: design updates
Parts:
- added D1: D_1A_30V_310mV, Diode_SMD:D_PowerDI-123, F.Cu at (155.4, 74.2)
- added D2: SMBJ5.0A, Diode_SMD:D_SMB, F.Cu at (130.2, 107.1)
- added D3: SMBJ5.0A, Diode_SMD:D_SMB, F.Cu at (160.2, 107.1)
- added J3: Conn_01x03, Connector_PinHeader_2.54mm:PinHeader_1x03_P2.54mm_Vertical, F.Cu at (128.0, 73.3)
- added R2: 150, Resistor_SMD:R_0603_1608Metric, F.Cu at (132.9, 73.5)
- added R3: 150, Resistor_SMD:R_0603_1608Metric, F.Cu at (119.3, 73.7)
- moved J1 0.08 mm to (122.0, 111.8)
Connections:
- C5 pad 1: +5V -> +3V3
- C6 pad 1: +5V -> +3V3
- U1 pad 17: Net-(U1-Pad17) -> +BATT
- U3 pad 6: +5V -> +3V3
- U4 pad 6: +5V -> +3V3
Routing:
- net +3V3: track 0.00 -> 71.7 mm
- net +BATT: track 0.00 -> 36.1 mm
- net +5V: track 53.0 -> 30.9 mm
- net +24V: track 82.8 -> 104.0 mm
- net Net-(R2-Pad1): track 0.00 -> 8.88 mm
- net GND: track 9.72 -> 18.4 mm
- net Net-(R3-Pad1): track 0.00 -> 7.72 mm
- net Net-(J3-Pad1): track 0.00 -> 4.25 mm
- net /SCL: track 41.0 -> 45.0 mm
- net Net-(J3-Pad3): track 0.00 -> 2.94 mm
- net Net-(D2-Pad1): track 15.3 -> 17.4 mm
- net Net-(D3-Pad1): track 24.1 -> 25.6 mm
- net /SDA: track 45.3 -> 45.9 mm

Commit message: start of gateway changes
Parts:
- removed D1: D_1A_30V_310mV, Diode_SMD:D_PowerDI-123
- added R4: 4.7K, Resistor_SMD:R_0603_1608Metric, F.Cu at (110.0, 99.8)
- added R5: 4.7K, Resistor_SMD:R_0603_1608Metric, F.Cu at (105.8, 99.8)
Connections:
- C5 pad 1: +3V3 -> +5V
- C6 pad 1: +3V3 -> +5V
- U3 pad 6: +3V3 -> +5V
- U4 pad 6: +3V3 -> +5V
Routing:
- net +5V: track 30.9 -> 52.6 mm
- net +3V3: track 71.7 -> 55.5 mm, vias 0 -> 2
- net /SDA: track 45.9 -> 48.2 mm
- net /SCL: track 45.0 -> 46.0 mm
