File: siot-gateway-particle-io/siot-gateway-particle-io.sch (KiCad schematic (older format))
At the start: 28 parts, among them J1 xConnect_smd, J2 xConnect_smd, J3 Conn_01x03, U1 Particle_Mesh, U2 LTC3630, U3 DS2483R, U4 DS2483R, U5 MDC3105LT1G, U6 MDC3105LT1G

Commit message: work on gw with IO
Parts:
- U5, U6: symbol bec-power:MDC3105LT1G -> siot-gateway-particle-io-rescue:MDC3105LT1G-bec-power
Changed lines of the file:
@@
 EESchema Schematic File Version 4
-LIBS:siot-gateway-particle-io-cache
 EELAYER 30 0
 EELAYER END
 $Descr USLetter 11000 8500
 encoding utf-8
-Sheet 1 1
+Sheet 1 2
 Title "SIoT Gateway (Particle) IO"
 Date "2019-08-20"
@@
 $EndComp
 $Comp
-L bec-power:MDC3105LT1G U5
+L siot-gateway-particle-io-rescue:MDC3105LT1G-bec-power U5
 U 1 1 5D805251
 P 8150 3750
@@
 $EndComp
 $Comp
-L bec-power:MDC3105LT1G U6
+L siot-gateway-particle-io-rescue:MDC3105LT1G-bec-power U6
 U 1 1 5D805889
 P 8200 4600
@@
 	1    0    0    -1
 $EndComp
+$Sheet
+S 8850 5850 1200 650
+U 5E6DB8BD
+F0 "Universal IO" 50
+F1 "sheet2.sch" 50
+$EndSheet
 $EndSCHEMATC
