File: rpi-odroid-expansion/rpi-odroid-expansion.sch (KiCad schematic (older format))
At the start: 17 parts, among them J1 RJ9, J2 RJ9, J3 Conn_02x20_Odd_Even, J4 RJ45, U1 DS2484R, U2 DS2484R, U3 PCF8563TS, U4 STM32F042K4Tx, U5 TSC2046, Y1 32.768KHz

Commit message: progress on board
Parts:
- added J5: RJ45, symbol Connector:RJ45
- added R1: 20, symbol Device:R_US
- added U6: MCP2551-I-SN, Package_SO:SOIC-8_3.9x4.9mm_P1.27mm, symbol Interface_CAN_LIN:MCP2551-I-SN
- added U7: MAX13487E, Package_SO:SO-8_3.9x4.9mm_P1.27mm, symbol bec-interface:MAX13487E
- BAT1: symbol dk_Battery-Holders-Clips-Contacts:BS-7 -> bec-connector:batt-2032
- gave numbers to parts that had none: 3
Connections:
- net labels added: CAN_RX, CAN_TX, GPIO1, GPIO2, GPIO3, GPIO4, GPIO5, LCD_DC, LCD_RSTn, RS485_RX, RS485_TX, X+, X-, Y+, Y-
- net labels removed: CAN_H, CAN_L
- wire segments 100 -> 221
Other:
- note added: "Backlight requires\n90mA @ ~3.2V\n(5v-3.2v)/90ma = ~20ohm"
- note added: "LCD Configured \nfor 8-bit, 4-wire\nSPI mode"
- note added: "Notes:\n1) TODO: add RS485 bias resistors\n2) TODO: add decoupling\n"
- note added: "RS485\nPort"
- moved on the sheet: BAT1, C1, D1, D2, J1, J2, J3, J4, J7, LCD1, U1, U2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

Commit message: add more notes
Other:
- note added: "Notes:\n1) TODO: add RS485 bias resistors\n2) TODO: add decoupling\n3) TODO: ISP for MCU (perhaps USB port)\n4) TODO: finialize connectors"
- note removed: "Notes:\n1) TODO: add RS485 bias resistors\n2) TODO: add decoupling\n"
Changed lines of the file:
@@
 Backlight requires\n90mA @ ~3.2V\n(5v-3.2v)/90ma = ~20ohm
 Text Notes 5950 5900 0    50   ~ 0
-Notes:\n1) TODO: add RS485 bias resistors\n2) TODO: add decoupling\n
+Notes:\n1) TODO: add RS485 bias resistors\n2) TODO: add decoupling\n3) TODO: ISP for MCU (perhaps USB port)\n4) TODO: finialize connectors
 $Comp
 L Device:R_US R1

Commit message: more notes/documentation
Other:
- note added: "Notes:\n1) TODO: add RS485 bias resistors\n2) TODO: add decoupling\n3) TODO: ISP for MCU (perhaps USB port)\n4) TODO: finialize connectors\n5) TODO: wire SPI from MPU to MCU\n6) TODO: bring out unused MPU/MCU pins to test points"
- note removed: "Notes:\n1) TODO: add RS485 bias resistors\n2) TODO: add decoupling\n3) TODO: ISP for MCU (perhaps USB port)\n4) TODO: finialize connectors"
Changed lines of the file:
@@
 Backlight requires\n90mA @ ~3.2V\n(5v-3.2v)/90ma = ~20ohm
 Text Notes 5950 5900 0    50   ~ 0
-Notes:\n1) TODO: add RS485 bias resistors\n2) TODO: add decoupling\n3) TODO: ISP for MCU (perhaps USB port)\n4) TODO: finialize connectors
+Notes:\n1) TODO: add RS485 bias resistors\n2) TODO: add decoupling\n3) TODO: ISP for MCU (perhaps USB port)\n4) TODO: finialize connectors\n5) TODO: wire SPI from MPU to MCU\n6) TODO: bring out unused MPU/MCU pins to test points
 $Comp
 L Device:R_US R1

Commit message: more notes and design tweaks
Connections:
- net labels added: GPIO12, GPIO13, GPIO18, GPIO19, GPIO22, GPIO23, GPIO24, GPIO25, GPIO26, GPIO27, GPIO6, MCU_RSTn, SPI_CS2
- wire segments 221 -> 238
Changed lines of the file:
@@
 $EndComp
-Wire Wire Line
-	1800 1500 1850 1500
 Wire Wire Line
 	1850 1500 1850 1900
@@
 $EndComp
 Wire Wire Line
-	3500 1600 2850 1600
-Wire Wire Line
-	3500 1850 2850 1850
-Text Label 2950 1600 0    50   ~ 0
+	3500 1600 3050 1600
+Wire Wire Line
+	3500 1850 3050 1850
+Text Label 3100 1600 0    50   ~ 0
 I2C_SDA
-Text Label 2950 1850 0    50   ~ 0
+Text Label 3100 1850 0    50   ~ 0
 I2C_SCL
 Wire Wire Line
-	3500 1350 2850 1350
-Text Label 2950 1350 0    50   ~ 0
+	3500 1350 3050 1350
+Text Label 3100 1350 0    50   ~ 0
 W1_BUSA
 Wire Wire Line
@@
 $EndComp
 Wire Wire Line
-	3500 2900 2850 2900
-Wire Wire Line
-	3500 3150 2850 3150
-Text Label 2950 2900 0    50   ~ 0
+	3500 2900 3050 2900
+Wire Wire Line
+	3500 3150 3050 3150
+Text Label 3100 2900 0    50   ~ 0
 I2C_SDA
-Text Label 2950 3150 0    50   ~ 0
+Text Label 3100 3150 0    50   ~ 0
 I2C_SCL
 Wire Wire Line
-	3500 2650 2850 2650
-Text Label 2950 2650 0    50   ~ 0
+	3500 2650 3050 2650
+Text Label 3100 2650 0    50   ~ 0
 W1_BUSA
 Wire Wire Line
@@
 	4250 3150 4250 3200
 Wire Wire Line
-	4200 1600 4700 1600
-Wire Wire Line
-	4200 2900 4750 2900
-Text Label 4350 1600 0    50   ~ 0
+	4200 1600 4500 1600
+Wire Wire Line
+	4200 2900 4550 2900
+Text Label 4250 1600 0    50   ~ 0
 W1_A
-Text Label 4400 2900 0    50   ~ 0
+Text Label 4300 2900 0    50   ~ 0
 W1_B
 $Comp
@@
 CAN_RX
 Wire Wire Line
-	6950 2450 7400 2450
-Wire Wire Line
-	6950 2350 7400 2350
+	6950 2450 7550 2450
+Wire Wire Line
+	6950 2350 7550 2350
 Text Label 7050 2450 0    50   ~ 0
 CAN_TX
@@
 	1800 2800 2400 2800
 Text Label 1950 2800 0    50   ~ 0
-LCD_RSTn
+GPIO12
 Wire Wire Line
 	8600 3300 9450 3300
@@
 Wire Wire Line
 	1800 3000 2400 3000
-Text Label 1950 3000 0    50   ~ 0
-LCD_DC
 $Comp
 L bec-interface:MAX13487E U7
@@
 	1300 3100 650  3100
 Text Label 700  2700 0    50   ~ 0
-GPIO1
+GPIO5
 Text Label 700  2800 0    50   ~ 0
-GPIO2
+GPIO6
 Text Label 700  2900 0    50   ~ 0
-GPIO3
+GPIO13
 Text Label 700  3000 0    50   ~ 0
-GPIO4
+GPIO19
 Text Label 700  3100 0    50   ~ 0
-GPIO5
+GPIO26
 Wire Wire Line
 	5300 2050 5950 2050
@@
 Wire Wire Line
 	9350 1600 9450 1600
+Wire Wire Line
+	1800 1600 2400 1600
+Text Label 1900 1600 0    50   ~ 0
+UART_TX
+Text Label 1900 1700 0    50   ~ 0
+UART_RX
+Wire Wire Line
+	1800 1700 2400 1700
+Wire Wire Line
+	1800 1500 1850 1500
+Wire Wire Line
+	1300 1900 650  1900
+Wire Wire Line
+	1300 2000 650  2000
+Text Label 750  1900 0    50   ~ 0
+GPIO27
+Text Label 750  2000 0    50   ~ 0
+GPIO22
+Wire Wire Line
+	1800 3100 2400 3100
+Wire Wire Line
+	1800 3200 2400 3200
+Text Label 1950 3100 0    50   ~ 0
+LCD_DC
+Text Label 1950 3200 0    50   ~ 0
+LCD_RSTn
+Wire Wire Line
+	1800 1800 2400 1800
+Wire Wire Line
+	1800 2000 2400 2000
+Wire Wire Line
+	1800 2100 2400 2100
+Wire Wire Line
+	1800 2300 2400 2300
+Text Label 1900 1800 0    50   ~ 0
+GPIO18
+Text Label 1950 2000 0    50   ~ 0
+GPIO23
+Text Label 1950 2100 0    50   ~ 0
+GPIO24
+Text Label 2050 2300 0    50   ~ 0
+GPIO25
+Wire Wire Line
+	6950 1750 7550 1750
+Wire Wire Line
+	6950 1850 7550 1850
+Wire Wire Line
+	6950 1950 7550 1950
+Text Label 7050 1750 0    50   ~ 0
+SPI_CLK
+Text Label 7050 1850 0    50   ~ 0
+SPI_MOSI
+Text Label 7050 1950 0    50   ~ 0
+SPI_MISO
+Wire Wire Line
+	5300 2550 5950 2550
+Text Label 5350 2550 0    50   ~ 0
+ID_SCL
+Wire Wire Line
+	5950 2650 5300 2650
+Text Label 5350 2650 0    50   ~ 0
+ID_SDA
+Text Label 1950 3000 0    50   ~ 0
+MCU_RSTn
+Wire Wire Line
+	5950 1250 5300 1250
+Text Label 5350 1250 0    50   ~ 0
+MCU_RSTn
+Wire Wire Line
+	6950 1650 7550 1650
+Text Label 7050 1650 0    50   ~ 0
+SPI_CS2
 $EndSCHEMATC

Commit message: fill in pn's, pull in rPI hat outline, etc
Parts:
- J1, J2: footprint (none) -> Connector_RJ:RJ12_Amphenol_54601
- J3: value Conn_02x20_Odd_Even -> rPI_02x20; footprint (none) -> Simple Iot:Samtec_HLE-120-02-XXX-DV-BE-XX-XX; symbol Connector_Generic:Conn_02x20_Odd_Even -> bec-connector:rPI_02x20; MPN (none) -> C25582-40G-M36-0A; Manufacturer (none) -> Kaweei
- J4, J5: footprint (none) -> Connector_RJ:RJ45_Amphenol_54602-x08_Horizontal
- U3: symbol Timer_RTC:PCF8563TS -> bec-interface:PCF8563TS; MPN (none) -> PCF8563TS/5; Manufacturer (none) -> NXP
- U4: value STM32F042K4Tx -> STM32F042K4T6; symbol MCU_ST_STM32F0:STM32F042K4Tx -> bec-cpu:STM32F042K4T6; MPN (none) -> STM32F042K4T6; Manufacturer (none) -> ST
- U5: MPN (none) -> TSC2046IPW; Manufacturer (none) -> TI
- U6: symbol Interface_CAN_LIN:MCP2551-I-SN -> bec-interface:MCP2551-I-SN; MPN (none) -> MCP2551-I/SN; Manufacturer (none) -> Microchip
- U7: MPN (none) -> MAX13487EESA+; Manufacturer (none) -> Maxim
Changed lines of the file:
@@
 	1250 3200 1250 3300
 $Comp
-L Connector_Generic:Conn_02x20_Odd_Even J3
+L bec-connector:rPI_02x20 J3
 U 1 1 5DF007AE
 P 1500 2200
 F 0 "J3" H 1550 3317 50  0000 C CNN
-F 1 "Conn_02x20_Odd_Even" H 1550 3226 50  0000 C CNN
-F 2 "" H 1500 2200 50  0001 C CNN
-F 3 "~" H 1500 2200 50  0001 C CNN
+F 1 "rPI_02x20" H 1550 3226 50  0000 C CNN
+F 2 "Simple Iot:Samtec_HLE-120-02-XXX-DV-BE-XX-XX" H 1500 2200 50  0001 C CNN
+F 3 "https://cdn-shop.adafruit.com/product-files/2187/CS25582-40G-M36-0A+(1).jpg" H 1500 2200 50  0001 C CNN
+F 4 "C25582-40G-M36-0A" H 1500 2200 50  0001 C CNN "MPN"
+F 5 "Kaweei" H 1500 2200 50  0001 C CNN "Manufacturer"
 	1    1500 2200
 	1    0    0    -1
@@
 F 0 "J1" H 1407 4667 50  0000 C CNN
 F 1 "RJ9" H 1407 4576 50  0000 C CNN
-F 2 "" V 1350 4250 50  0001 C CNN
+F 2 "Connector_RJ:RJ12_Amphenol_54601" V 1350 4250 50  0001 C CNN
 F 3 "~" V 1350 4250 50  0001 C CNN
 	1    1350 4200
@@
 F 0 "J2" H 1407 5717 50  0000 C CNN
 F 1 "RJ9" H 1407 5626 50  0000 C CNN
-F 2 "" V 1350 5300 50  0001 C CNN
+F 2 "Connector_RJ:RJ12_Amphenol_54601" V 1350 5300 50  0001 C CNN
 F 3 "~" V 1350 5300 50  0001 C CNN
 	1    1350 5250
@@
 W1_B
 $Comp
-L Timer_RTC:PCF8563TS U3
+L bec-interface:PCF8563TS U3
 U 1 1 5DF1C663
 P 3850 5100
@@
 F 1 "PCF8563TS" H 4100 5450 50  0000 C CNN
 F 2 "Package_SO:MSOP-8_3x3mm_P0.65mm" H 3850 5100 50  0001 C CNN
-F 3 "https://assets.nexperia.com/documents/data-sheet/PCF8563.pdf" H 3850 5100 50  0001 C CNN
+F 3 "https://www.nxp.com/docs/en/data-sheet/PCF8563.pdf" H 3850 5100 50  0001 C CNN
+F 4 "PCF8563TS/5" H 3850 5100 50  0001 C CNN "MPN"
+F 5 "NXP" H 3850 5100 50  0001 C CNN "Manufacturer"
 	1    3850 5100
 	1    0    0    -1
@@
 SPI_CS1
 $Comp
-L MCU_ST_STM32F0:STM32F042K4Tx U4
+L bec-cpu:STM32F042K4T6 U4
 U 1 1 5F6D1E5B
 P 6450 1950
 F 0 "U4" H 6600 900 50  0000 C CNN
-F 1 "STM32F042K4Tx" H 6850 1000 50  0000 C CNN
+F 1 "STM32F042K4T6" H 6850 1000 50  0000 C CNN
 F 2 "Package_QFP:LQFP-32_7x7mm_P0.8mm" H 6050 1050 50  0001 R CNN
 F 3 "http://www.st.com/st-web-ui/static/active/en/resource/technical/document/datasheet/DM00105814.pdf" H 6450 1950 50  0001 C CNN
+F 4 "STM32F042K4T6" H 6450 1950 50  0001 C CNN "MPN"
+F 5 "ST" H 6450 1950 50  0001 C CNN "Manufacturer"
 	1    6450 1950
 	1    0    0    -1
@@
 F 0 "J4" H 1020 6304 50  0000 R CNN
 F 1 "RJ45" H 1020 6395 50  0000 R CNN
-F 2 "" V 1350 6325 50  0001 C CNN
+F 2 "Connector_RJ:RJ45_Amphenol_54602-x08_Horizontal" V 1350 6325 50  0001 C CNN
 F 3 "~" V 1350 6325 50  0001 C CNN
 	1    1350 6300
@@
 F 2 "Package_SO:SSOP-16_3.9x4.9mm_P0.635mm" H 6400 3600 50  0001 C CIN
 F 3 "https://www.ti.com/lit/ds/symlink/tsc2046.pdf" H 6600 3650 50  0001 C CNN
+F 4 "TSC2046IPW" H 6400 4200 50  0001 C CNN "MPN"
+F 5 "TI" H 6400 4200 50  0001 C CNN "Manufacturer"
 	1    6400 4200
 	1    0    0    -1
@@
 Y-
 $Comp
-L Interface_CAN_LIN:MCP2551-I-SN U6
+L bec-interface:MCP2551-I-SN U6
 U 1 1 5F763739
 P 3450 6400
@@
 F 2 "Package_SO:SOIC-8_3.9x4.9mm_P1.27mm" H 3450 5900 50  0001 C CIN
 F 3 "http://ww1.microchip.com/downloads/en/devicedoc/21667d.pdf" H 3450 6400 50  0001 C CNN
+F 4 "MCP2551-I/SN" H 3450 6400 50  0001 C CNN "MPN"
+F 5 "Microchip" H 3450 6400 50  0001 C CNN "Manufacturer"
 	1    3450 6400
 	-1   0    0    -1
@@
 F 2 "Package_SO:SO-8_3.9x4.9mm_P1.27mm" H 3650 7900 50  0001 C CNN
 F 3 "https://datasheets.maximintegrated.com/en/ds/MAX13487E-MAX13488E.pdf" H 3650 7900 50  0001 C CNN
+F 4 "Maxim" H 3650 7900 50  0001 C CNN "Manufacturer"
+F 5 "MAX13487EESA+" H 3650 7900 50  0001 C CNN "MPN"
 	1    3650 7900
 	-1   0    0    -1
@@
 F 0 "J5" H 1020 7404 50  0000 R CNN
 F 1 "RJ45" H 1020 7495 50  0000 R CNN
-F 2 "" V 1350 7425 50  0001 C CNN
+F 2 "Connector_RJ:RJ45_Amphenol_54602-x08_Horizontal" V 1350 7425 50  0001 C CNN
 F 3 "~" V 1350 7425 50  0001 C CNN
 	1    1350 7400
